Commit message: añadimos restricciones de rotación en las ruedas diferenciales y añadimos base footprint

File: session2/myrobot_1.urdf (robot description, URDF)
Before this commit: robot myrobot_1, 4 links, 3 joints
Links:
- added link base_footprint
Joints:
- added joint base_joint: type fixed, parent base_footprint, child base_link, origin xyz=0 0 0 rpy=0 0 0, axis 0 0 0
- joint base_caster_wheel_joint: axis (none) -> 0 0 0; type continuous -> fixed
- joint base_left_wheel_joint: axis (none) -> 0 1 0
- joint base_right_wheel_joint: axis (none) -> 0 1 0

Commit message: un arreglillo

File: session2/myrobot_1.urdf (robot description, URDF)
Before this commit: robot myrobot_1, 5 links, 4 joints
Joints:
- joint base_caster_wheel_joint: origin xyz=0.15 0 0.1 rpy=0 0 0 -> xyz=0.15 0 -0.1 rpy=0 0 0
- joint base_joint: origin xyz=0 0 0 rpy=0 0 0 -> xyz=0 0 0.2 rpy=0 0 0
- joint base_left_wheel_joint: origin xyz=-0.15 0.2 0.1 rpy=0 0 0 -> xyz=-0.15 0.2 -0.1 rpy=0 0 0
- joint base_right_wheel_joint: origin xyz=-0.15 -0.2 0.1 rpy=0 0 0 -> xyz=-0.15 -0.2 -0.1 rpy=0 0 0
