Commit message: Sessio4 acabado

File: session3/myrobot_1_description/urdf/myrobot_1.urdf (robot description, URDF)
Before this commit: robot myrobot_1, 5 links, 4 joints
Links:
- added link imu; collision box size=0.05 0.05 0.02; visual box size=0.05 0.05 0.02
- added link lidar; collision cylinder length=0.05 radius=0.06; visual cylinder length=0.05 radius=0.06
Joints:
- added joint base_imu_joint: type fixed, parent base_link, child imu, origin xyz=0 0 -0.1 rpy=0 0 0, axis 0 0 0
- added joint base_lidar_joint: type fixed, parent base_link, child lidar, origin xyz=0 0 0.1 rpy=0 0 0, axis 0 0 0
